Commit message: Added documentation in regards to accessing camera data via rqt. Added textures for the tasks, hopefully stonefish will support these in the near future.

File: tardigrade/metadata/looks.scn.xacro (robot description, xacro)
@@ -10,4 +10,5 @@
     <looks>
         <look name="black" gray="0.05" roughness="0.2"/>
+        <look name="orange" rgb="1.0 0.35 0.0" roughness="0.2"/>
         <look name="yellow" rgb="1.0 0.9 0.0" roughness="0.3"/>
         <look name="blue" rgb="0.1 0.1 0.9" roughness="0.3"/>
@@ -15,9 +16,10 @@
         <look name="gray" gray="0.5" roughness="0.4" metalness="0.5"/>
         <look name="tank" rgb="0.9 0.9 0.9" roughness="0.9"/>
-        <look name="ice" rgb="0.31 0.34 0.35" roughness="0.9"/>
         <look name="duct" gray="0.1" roughness="0.4" metalness="0.5"/>
-        <look name="manipulator" rgb="0.2 0.15 0.1" roughness="0.6" metalness="0.8"/>
-        <look name="ee" rgb="0.59 0.56 0.51" roughness="0.6" metalness="0.8"/>
         <look name="green" rgb="0.0 1.0 0.0" roughness="0.5" metalness="0.1"/>
+        <look name="white" gray="0.95" roughness="0.2"/>
+        <look name="buoy" gray="0.1" roughness="0.1" texture="$(find tardigrade)/data/BuoyTexture.jpg"/>
+        <look name="gate" gray="0.1" roughness="0.1" texture="$(find tardigrade)/data/GateTexture.jpg"/>
+        <look name="path" gray="0.1" roughness="0.1" texture="$(find tardigrade)/data/PathTexture.jpg"/>
     </looks>
 </scenario>

File: tardigrade/vehicles/tardigrade.scn.xacro (robot description, xacro)
@@ -118,5 +118,5 @@
 						<ros_subscriber topic = "/${robot_name}/control/thruster/starboard_surge"/>
 					</actuator>
-					<sensor name="IMU" type="imu" rate="20.0">
+					<sensor name="IMU" type="imu" rate="10.0">
 						<link name="Base"/>
 						<origin rpy = "0.0 0.0 0.0" xyz = "0.0 0.0 0.0"/>
@@ -124,16 +124,28 @@
 						<ros_publisher topic="/${robot_name}/imu/stonefish/data"/>
 					</sensor>
-					<sensor name="CameraFront" rate="10.0" type="camera">
+					<sensor name="CameraFront" rate="1.0" type="camera">
 						<specs resolution_x="1920" resolution_y="1080" horizontal_fov="150"/>
-						<origin rpy="4.7124 0.0 -1.571" xyz="0.355749 0.0 -0.139725"/>
+						<origin rpy="1.5708 0.0 1.5708" xyz="0.355749 0.0 -0.139725"/>
 						<link name="Base"/>
 						<ros_publisher topic="/${robot_name}/camera/stonefish/front/data"/>
 					</sensor>
-					<sensor name="CameraTop" rate="10.0" type="camera">
-						<specs resolution_x="640" resolution_y="480" horizontal_fov="180"/>
-						<origin rpy="4.7124 3.1416 -1.571" xyz="0.0 0.0 1.5"/>
+					<sensor name="CameraTop" rate="1.0" type="camera">
+						<specs resolution_x="1080" resolution_y="1080" horizontal_fov="175"/>
+						<origin rpy="0.0 3.14159 1.5708" xyz="0.0 0.0 -0.1"/>
 						<link name="Base"/>
 						<ros_publisher topic="/${robot_name}/camera/stonefish/top/data"/>
 					</sensor>
+                    <light name="spotlightA">
+                        <specs radius="0.1" cone_angle="30.0" illuminance="2000.0"/>
+                        <color temperature="5600.0"/>
+                        <origin rpy="4.7124 0.0 -1.571" xyz="0.355749 0.25 -0.139725"/>
+                        <link name="Base"/>
+                    </light>
+                    <light name="spotlightB">
+                        <specs radius="0.1" cone_angle="30.0" illuminance="2000.0"/>
+                        <color temperature="5600.0"/>
+                        <origin rpy="4.7124 0.0 -1.571" xyz="0.355749 -0.25 -0.139725"/>
+                        <link name="Base"/>
+                    </light>
 			<world_transform rpy="${rpy}" xyz="${xyz}"/>
         </robot>

File: tardigrade/world/tank.scn.xacro (robot description, xacro)
@@ -8,19 +8,19 @@
     <xacro:arg name="robot_name" default="tardigrade"/>
     <xacro:include filename="$(find tardigrade)/vehicles/$(arg robot_name).scn.xacro"/>
-    <xacro:tardigrade robot_name="$(arg robot_name)" xyz="0.0 0.0 0.0" rpy="0.0 0.0 0.0"/>
+    <xacro:tardigrade robot_name="$(arg robot_name)" xyz="0.0 20.0 0.0" rpy="0.0 0.0 0.0"/>
     <environment>
         <ned latitude="0" longitude="0"/>
         <ocean>
-            <water density="1000.0" jerlov="0.2"/>
+            <water density="1031.0" jerlov="0.2"/>
             <waves height="0.0"/>
             <particles enabled="true"/>
             <current type="uniform">
+                <velocity xyz="1.0 0.0 0.0"/>
+            </current>
+            <current type="jet">
+                <center xyz="0.0 0.0 3.0"/>
+                <outlet radius="0.0"/>
                 <velocity xyz="0.0 0.0 0.0"/>
             </current>
-            <!-- <current type="jet">
-                <center xyz="0.0 0.0 3.0"/>
-                <outlet radius="0.2"/>
-                <velocity xyz="0.0 2.0 0.0"/>
-            </current> -->
         </ocean>
         <atmosphere>
@@ -41,3 +41,42 @@
         <world_transform xyz="0.0 0.0 4.0" rpy="3.1415926 0.0 0.0"/>
     </static>
+    <static name="gate" type="model">
+        <physical>
+            <mesh filename="$(find tardigrade)/data/objects/Gate.obj" scale="0.001"/>
+            <origin xyz="0.0 0.0 0.0" rpy="0.0 0.0 0.0"/>
+        </physical>
+        <visual>
+            <mesh filename="$(find tardigrade)/data/objects/Gate.obj" scale="0.001"/>
+            <origin xyz="0.0 0.0 0.0" rpy="0.0 0.0 0.0"/>
+        </visual>
+        <material name="Neutral"/>"
+        <look name="gray"/>
+        <world_transform xyz="0.0 0.0 2.5" rpy="0.0 0.0 0.0"/>
+    </static>
+    <static name="buoy" type="model">
+        <physical>
+            <mesh filename="$(find tardigrade)/data/objects/Buoy.obj" scale="0.001"/>
+            <origin xyz="0.0 0.0 0.0" rpy="0.0 0.0 0.0"/>
+        </physical>
+        <visual>
+            <mesh filename="$(find tardigrade)/data/objects/Buoy.obj" scale="0.001"/>
+            <origin xyz="0.0 0.0 0.0" rpy="0.0 0.0 0.0"/>
+        </visual>
+        <material name="Neutral"/>
+        <look name="red"/>
+        <world_transform xyz="0.0 0.0 1.0" rpy="0.0 3.14159 0.0"/>
+    </static>
+    <static name="path" type="model">
+        <physical>
+            <mesh filename="$(find tardigrade)/data/objects/Path.obj" scale="0.001"/>
+            <origin xyz="0.0 0.0 0.0" rpy="0.0 0.0 0.0"/>
+        </physical>
+        <visual>
+            <mesh filename="$(find tardigrade)/data/objects/Path.obj" scale="0.001"/>
+            <origin xyz="0.0 0.0 0.0" rpy="0.0 0.0 0.0"/>
+        </visual>
+        <material name="Neutral"/>
+        <look name="orange"/>
+        <world_transform xyz="0.0 0.0 2.5" rpy="0.0 0.0 0.0"/>
+    </static>
 </scenario>
