Commit message: Added alot more seperation for the purpose of containerizing our surface ROS packages, and our onboard packages. I also changed the package names as we will just use the same one, and just change the mission order.

File: tardigrade/vehicles/tardigrade.scn.xacro (robot description, xacro)
@@ -7,6 +7,6 @@
 -->
 <scenario xmlns:xacro="http://ros.org/wiki/xacro">
-    <xacro:include filename = "$(find prequal)/metadata/looks.scn.xacro"/>
-    <xacro:include filename = "$(find prequal)/metadata/materials.scn.xacro"/>
+    <xacro:include filename = "$(find tardigrade)/metadata/looks.scn.xacro"/>
+    <xacro:include filename = "$(find tardigrade)/metadata/materials.scn.xacro"/>
 	<xacro:macro name = "tardigrade" params = "xyz rpy robot_name">
 	<!--Shell Generator-->

File: tardigrade/world/prequal_tank.scn.xacro (robot description, xacro)
@@ -7,5 +7,5 @@
 <scenario xmlns:xacro="http://ros.org/wiki/xacro">
     <xacro:arg name="robot_name" default="tardigrade"/>
-    <xacro:include filename="$(find prequal)/vehicles/$(arg robot_name).scn.xacro"/>
+    <xacro:include filename="$(find tardigrade)/vehicles/$(arg robot_name).scn.xacro"/>
     <xacro:tardigrade robot_name="$(arg robot_name)" xyz="0.0 0.0 0.0" rpy="0.0 0.0 0.0"/>
     <environment>
@@ -30,9 +30,9 @@
     <static name="tank" type="model">
         <physical>
-            <mesh filename="$(find prequal)/data/objects/prequaltank.obj" scale="100.0"/>
+            <mesh filename="$(find tardigrade)/data/objects/prequaltank.obj" scale="100.0"/>
             <origin xyz="0.0 0.0 0.0" rpy="0.0 0.0 0.0"/>
         </physical>
         <visual>
-            <mesh filename="$(find prequal)/data/objects/prequaltank.obj" scale="100.0"/>
+            <mesh filename="$(find tardigrade)/data/objects/prequaltank.obj" scale="100.0"/>
             <origin xyz="0.0 0.0 0.0" rpy="0.0 0.0 0.0"/>
         </visual>

Commit message: Changed power output of thruster values to have a more controlled descent. Will need to computer forces to equalize the bow and stern thrusters.

File: tardigrade/vehicles/tardigrade.scn.xacro (robot description, xacro)
@@ -126,11 +126,11 @@
 					<sensor name="CameraFront" rate="1.0" type="camera">
 						<specs resolution_x="1920" resolution_y="1080" horizontal_fov="150"/>
-						<origin rpy="1.5708 0.0 1.5708" xyz="0.355749 0.0 -0.139725"/>
+						<origin rpy="1.5708 0.0 1.5708" xyz="0.38 0.0 -0.15"/>
 						<link name="Base"/>
 						<ros_publisher topic="/${robot_name}/camera/stonefish/front/data"/>
 					</sensor>
 					<sensor name="CameraTop" rate="1.0" type="camera">
-						<specs resolution_x="1080" resolution_y="1080" horizontal_fov="175"/>
-						<origin rpy="0.0 3.14159 1.5708" xyz="0.0 0.0 -0.1"/>
+						<specs resolution_x="640" resolution_y="640" horizontal_fov="179"/>
+						<origin rpy="0.0 3.14159 1.5708" xyz="0.0 0.0 -0.15"/>
 						<link name="Base"/>
 						<ros_publisher topic="/${robot_name}/camera/stonefish/top/data"/>

Commit message: Robot go brr

File: tardigrade/vehicles/tardigrade.scn.xacro (robot description, xacro)
@@ -126,26 +126,32 @@
 					<sensor name="CameraFront" rate="10.0" type="camera">
 						<specs resolution_x="1920" resolution_y="1080" horizontal_fov="150"/>
-						<origin rpy="1.5708 0.0 1.5708" xyz="0.38 0.0 -0.15"/>
+						<origin rpy="1.5708 0.0 1.5708" xyz="0.38 0.0 -0.11"/>
 						<link name="Base"/>
-						<ros_publisher topic="/${robot_name}/camera/stonefish/front/data"/>
+						<ros_publisher topic="/${robot_name}/camera/front/data"/>
 					</sensor>
 					<sensor name="CameraTop" rate="5.0" type="camera">
 						<specs resolution_x="640" resolution_y="640" horizontal_fov="179"/>
-						<origin rpy="0.0 3.14159 1.5708" xyz="0.0 0.0 -0.15"/>
+						<origin rpy="0.0 3.14159 1.5708" xyz="0.0 0.0 -0.11"/>
 						<link name="Base"/>
-						<ros_publisher topic="/${robot_name}/camera/stonefish/top/data"/>
+						<ros_publisher topic="/${robot_name}/camera/top/data"/>
 					</sensor>
-                    <light name="spotlightA">
-                        <specs radius="0.1" cone_angle="30.0" illuminance="2000.0"/>
-                        <color temperature="5600.0"/>
-                        <origin rpy="4.7124 0.0 -1.571" xyz="0.355749 0.25 -0.139725"/>
+                    <sensor name="FFEchosounder" rate="1.0" type="multibeam">
+                        <specs fov="30.0" steps="1"/>
+                        <range distance_min="0.5" distance_max="30.0"/>
+                        <noise distance="0.1"/>
+                        <history samples="1"/>
+						<origin rpy="0.0 0.0 0.0" xyz="0.38 0.0 -0.11"/>
                         <link name="Base"/>
-                    </light>
-                    <light name="spotlightB">
-                        <specs radius="0.1" cone_angle="30.0" illuminance="2000.0"/>
-                        <color temperature="5600.0"/>
-                        <origin rpy="4.7124 0.0 -1.571" xyz="0.355749 -0.25 -0.139725"/>
+                        <ros_publisher topic="/${robot_name}/echosounder/front/data"/>
+                    </sensor>
+                    <sensor name="DFEchosounder" rate="1.0" type="multibeam">
+                        <specs fov="30.0" steps="1"/>
+                        <range distance_min="0.5" distance_max="30.0"/>
+                        <noise distance="0.1"/>
+                        <history samples="1"/>
+						<origin rpy="0.0 4.7124 0.0" xyz="0.0 0.0 0.11"/>
                         <link name="Base"/>
-                    </light>
+                        <ros_publisher topic="/${robot_name}/echosounder/down/data"/>
+                    </sensor>
 			<world_transform rpy="${rpy}" xyz="${xyz}"/>
         </robot>
